Commit message: pre_final

File: src/combined_description/urdf/combined_robot.urdf.xacro (robot description, xacro)
@@ -8,6 +8,8 @@
     <xacro:motoman_gp7 prefix="gp7_"/>
     <!-- Define a fixed joint between Kiwi Cell and Motoman GP7 -->
+    <!-- Adjust the xyz and rpy values based on the correct alignment -->
     <joint name="kiwi_to_gp7" type="fixed">
-        <origin xyz="0 0 1" rpy="0 0 0"/>
+        <!-- Assume the GP7 base link needs to be lowered by 1 meter to align with Kiwi Cell -->
+        <origin xyz="0 0 0" rpy="0 0 3.15"/> <!-- Set xyz to 0 0 0 for direct alignment -->
         <parent link="kiwi_robot_base_plate_link"/>
         <child link="gp7_base_link"/>

File: src/kiwi_cell_description/urdf/kiwi_cell.urdf.xacro (robot description, xacro)
@@ -49,5 +49,5 @@
     <inertial>
       <origin
-        xyz="0 0 -0.008"
+        xyz="0 0 -2"
         rpy="0 0 0" />
       <mass
@@ -89,5 +89,5 @@
     type="fixed">
     <origin
-      xyz="0.875 0.5225 0.982"
+      xyz="1.2 0.5225 0.982"
       rpy="0 0 0" />
     <parent

Commit message: Gripper addition and robot base plate update

File: src/combined_description/urdf/combined_robot.urdf.xacro (robot description, xacro)
@@ -7,4 +7,11 @@
     <xacro:include filename="$(find motoman_gp7_description)/urdf/gp7_macro.xacro"/>
     <xacro:motoman_gp7 prefix="gp7_"/>
+    <!-- Include the Robotiq 2f 85 Gripper description -->
+    <xacro:include filename="$(find robotiq_2f_85_gripper_visualization)/urdf/robotiq_arg2f_85_model.xacro"/>
+<!--
+    <xacro:include filename="$(find combined_description)/urdf/base_plate.xacro"/>
+    <xacro:base_plate prefix="" parent="world">
+        <origin xyz="0 -0.05 ${0.015+0.010}" rpy="0 -${pi/2} ${pi/2}"/>
+    </xacro:base_plate> -->
     <!-- Define a fixed joint between Kiwi Cell and Motoman GP7 -->
     <!-- Adjust the xyz and rpy values based on the correct alignment -->
@@ -15,3 +22,10 @@
         <child link="gp7_base_link"/>
     </joint>
+    <!-- Define a fixed joint between Motoman GP7 and Gripper -->
+    <joint name="gp7_to_gripper" type="fixed">
+        <!-- Set the origin to match the physical placement of the gripper on the GP7 tool -->
+        <origin xyz="0 0 0" rpy="0 0 0"/> <!-- Adjust xyz and rpy based on alignment -->
+        <parent link="gp7_tool0"/>  <!-- Motoman GP7's end-effector link -->
+        <child link="robotiq_arg2f_base_link"/> <!-- Gripper's base link -->
+    </joint>
 </robot>

File: src/kiwi_cell_description/urdf/kiwi_cell.urdf.xacro (robot description, xacro)
@@ -89,5 +89,5 @@
     type="fixed">
     <origin
-      xyz="1.125 0.5225 0.982"
+      xyz="1.1 0.5 0.982"
       rpy="0 0 0" />
     <parent

Commit message: updated combined urdf

File: src/combined_description/urdf/combined_robot.urdf.xacro (robot description, xacro)
@@ -9,9 +9,4 @@
     <!-- Include the Robotiq 2f 85 Gripper description -->
     <xacro:include filename="$(find robotiq_2f_85_gripper_visualization)/urdf/robotiq_arg2f_85_model.xacro"/>
-<!--
-    <xacro:include filename="$(find combined_description)/urdf/base_plate.xacro"/>
-    <xacro:base_plate prefix="" parent="world">
-        <origin xyz="0 -0.05 ${0.015+0.010}" rpy="0 -${pi/2} ${pi/2}"/>
-    </xacro:base_plate> -->
     <!-- Define a fixed joint between Kiwi Cell and Motoman GP7 -->
     <!-- Adjust the xyz and rpy values based on the correct alignment -->
